File: hardware/schematic/mcu.kicad_sch (KiCad schematic)
At the start: 14 parts, among them Q1 AO3401A, SW1 SW_BOOT, U1 MIMXRT1062DVL6B, Y1 24MHz 12pF, Y2 32.768kHz 12.5pF

Commit message: PM review fixes: boot R_S, C51, decap note, notes, BOM fields
- MUST: add R22 (R_S) 1k 0402 0402WGF1001TCE / C11702 between Q1 drain
  (pin 3, new net BOOT_MODE0_Q) and BOOT_MODE0 (F11)
- C51 VBUS bulk 10uF 0603 -> 4.7uF 0402 (CL05A475MP5NRNC / C23733)
- docs/decisions.md: keep C11/C12; VDD_SOC total 32.5uF vs HDG ~33uF
- U3 description and root note: buck inductor is L1 (was "L2")
- mcu sheet note: WAKEUP (L6) / ONOFF (M6) rely on internal 100k PU
- APS6404L-3SQR-ZR pinout + USON-8 footprint checked vs AP Memory
  datasheet Rev 2.3 (no change); GPIO_SD_B0_04 ALT4 = FLEXSPIB_SS0_B
  confirmed in SDK fsl_iomuxc.h (H2 per DS Table 83)
- J3 TC2030 and TP1-TP5: MPN/LCSC "N/A - footprint only" + BOM_Note
- gen.py: reuse UUIDs from existing files (stable diffs), runs in-repo;
  netlist.json ignored
- kicad-cli sch erc: 0 errors, 0 warnings

Fixes #8
Parts:
- added R22: 1k, Resistor_SMD:R_0402_1005Metric, symbol TokenKey:R
Connections:
- net BOOT_MODE0: now also R22.2; no longer Q1.3 (D)
- new net BOOT_MODE0_Q: Q1.3 (D), R22.1
Other:
- note added: "WAKEUP (L6) and ONOFF (M6) are left unconnected and rely on their internal 100k pull-ups (IMXRT1060CEC Rev 4 Table 83: reset and default state Input, 100K PU). ONOFF also on TP5."
Changed lines of the file:
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@@
 (global_label "BOOT_MODE0" (shape passive) (at 157.48 198.12 180) (fields_autoplaced yes) (effects (font (size 1.27 1.27)) (justify right)) (property "Intersheetrefs" "${INTERSHEET_REFS}" (at 157.48 198.12 0) (effects (font (size 1.27 1.27)) (hide yes))))
 (global_label "GND" (shape passive) (at 167.64 198.12 0) (fields_autoplaced yes) (effects (font (size 1.27 1.27)) (justify left)) (property "Intersheetrefs" "${INTERSHEET_REFS}" (at 167.64 198.12 0) (effects (font (size 1.27 1.27)) (hide yes))))
-(symbol (lib_id "TokenKey:AO3401A") (at 165.10 215.90 0) (unit 1) (exclude_from_sim no) (in_bom yes) (on_board yes) (dnp no) (property "Reference" "Q1" (at 165.10 212.09 0) (effects (font (size 1.27 1.27)))) (property "Value" "AO3401A" (at 165.10 222.25 0) (effects (font (size 1.27 1.27)))) (property "Footprint" "Package_TO_SOT_SMD:SOT-23" (at 165.10 224.79 0) (effects (font (size 1.27 1.27)) (hide yes))) (property "Datasheet" "" (at 165.10 215.90 0) (effects (font (size 1.27 1.27)) (hide yes))) (property "Description" "Press SW_BOOT: BM1=0 and Q1 on => BM0=1 => mode 01 serial downloader" (at 165.10 215.90 0) (effects (font (size 1.27 1.27)) (hide yes))) (property "MPN" "AO3401A" (at 165.10 215.90 0) (effects (font (size 1.27 1.27)) (hide yes))) (property "LCSC" "C15127" (at 165.10 215.90 0) (effects (font (size 1.27 1.27)) (hide yes))) (pin "1") (pin "2") (pin "3") (instances (project "TokenKey-RT" (path "/69bcae8e-63e2-488c-b267-fe4af22cfb6e/23672d8f-53fc-4309-8a86-d888b8c0a089" (reference "Q1") (unit 1)))))
+(symbol (lib_id "TokenKey:AO3401A") (at 165.10 215.90 0) (unit 1) (exclude_from_sim no) (in_bom yes) (on_board yes) (dnp no) (property "Reference" "Q1" (at 165.10 212.09 0) (effects (font (size 1.27 1.27)))) (property "Value" "AO3401A" (at 165.10 222.25 0) (effects (font (size 1.27 1.27)))) (property "Footprint" "Package_TO_SOT_SMD:SOT-23" (at 165.10 224.79 0) (effects (font (size 1.27 1.27)) (hide yes))) (property "Datasheet" "" (at 165.10 215.90 0) (effects (font (size 1.27 1.27)) (hide yes))) (property "Description" "Press SW_BOOT: BM1=0 and Q1 on => BM0=1 (via R_S) => mode 01 serial downloader" (at 165.10 215.90 0) (effects (font (size 1.27 1.27)) (hide yes))) (property "MPN" "AO3401A" (at 165.10 215.90 0) (effects (font (size 1.27 1.27)) (hide yes))) (property "LCSC" "C15127" (at 165.10 215.90 0) (effects (font (size 1.27 1.27)) (hide yes))) (pin "1") (pin "2") (pin "3") (instances (project "TokenKey-RT" (path "/69bcae8e-63e2-488c-b267-fe4af22cfb6e/23672d8f-53fc-4309-8a86-d888b8c0a089" (reference "Q1") (unit 1)))))
 (global_label "BOOT_MODE1" (shape passive) (at 157.48 215.90 180) (fields_autoplaced yes) (effects (font (size 1.27 1.27)) (justify right)) (property "Intersheetrefs" "${INTERSHEET_REFS}" (at 157.48 215.90 0) (effects (font (size 1.27 1.27)) (hide yes))))
 (global_label "3V3" (shape passive) (at 172.72 215.90 0) (fields_autoplaced yes) (effects (font (size 1.27 1.27)) (justify left)) (property "Intersheetrefs" "${INTERSHEET_REFS}" (at 172.72 215.90 0) (effects (font (size 1.27 1.27)) (hide yes))))
-(global_label "BOOT_MODE0" (shape passive) (at 172.72 218.44 0) (fields_autoplaced yes) (effects (font (size 1.27 1.27)) (justify left)) (property "Intersheetrefs" "${INTERSHEET_REFS}" (at 172.72 218.44 0) (effects (font (size 1.27 1.27)) (hide yes))))
+(global_label "BOOT_MODE0_Q" (shape passive) (at 172.72 218.44 0) (fields_autoplaced yes) (effects (font (size 1.27 1.27)) (justify left)) (property "Intersheetrefs" "${INTERSHEET_REFS}" (at 172.72 218.44 0) (effects (font (size 1.27 1.27)) (hide yes))))
 (symbol (lib_id "TokenKey:SW_Push") (at 162.56 236.22 0) (unit 1) (exclude_from_sim no) (in_bom yes) (on_board yes) (dnp no) (property "Reference" "SW1" (at 162.56 232.41 0) (effects (font (size 1.27 1.27)))) (property "Value" "SW_BOOT" (at 162.56 240.03 0) (effects (font (size 1.27 1.27)))) (property "Footprint" "Button_Switch_SMD:SW_SPST_B3U-1000P" (at 162.56 242.57 0) (effects (font (size 1.27 1.27)) (hide yes))) (property "Datasheet" "" (at 162.56 236.22 0) (effects (font (size 1.27 1.27)) (hide yes))) (property "Description" "Bottom side" (at 162.56 236.22 0) (effects (font (size 1.27 1.27)) (hide yes))) (property "MPN" "B3U-1000P" (at 162.56 236.22 0) (effects (font (size 1.27 1.27)) (hide yes))) (property "LCSC" "C231329" (at 162.56 236.22 0) (effects (font (size 1.27 1.27)) (hide yes))) (pin "1") (pin "2") (instances (project "TokenKey-RT" (path "/69bcae8e-63e2-488c-b267-fe4af22cfb6e/23672d8f-53fc-4309-8a86-d888b8c0a089" (reference "SW1") (unit 1)))))
 (global_label "BOOT_MODE1" (shape passive) (at 157.48 236.22 180) (fields_autoplaced yes) (effects (font (size 1.27 1.27)) (justify right)) (property "Intersheetrefs" "${INTERSHEET_REFS}" (at 157.48 236.22 0) (effects (font (size 1.27 1.27)) (hide yes))))
 (global_label "GND" (shape passive) (at 167.64 236.22 0) (fields_autoplaced yes) (effects (font (size 1.27 1.27)) (justify left)) (property "Intersheetrefs" "${INTERSHEET_REFS}" (at 167.64 236.22 0) (effects (font (size 1.27 1.27)) (hide yes))))
+(symbol (lib_id "TokenKey:R") (at 162.56 254.00 0) (unit 1) (exclude_from_sim no) (in_bom yes) (on_board yes) (dnp no) (property "Reference" "R22" (at 162.56 250.19 0) (effects (font (size 1.27 1.27)))) (property "Value" "1k" (at 162.56 257.81 0) (effects (font (size 1.27 1.27)))) (property "Footprint" "Resistor_SMD:R_0402_1005Metric" (at 162.56 260.35 0) (effects (font (size 1.27 1.27)) (hide yes))) (property "Datasheet" "" (at 162.56 254.00 0) (effects (font (size 1.27 1.27)) (hide yes))) (property "Description" "R_S: series 1k Q1 drain -> BOOT_MODE0 (F11); limits current if F11 is driven as GPIO. Q1 on: BM0 = 3.3*10k/11k = 3.0 V" (at 162.56 254.00 0) (effects (font (size 1.27 1.27)) (hide yes))) (property "MPN" "0402WGF1001TCE" (at 162.56 254.00 0) (effects (font (size 1.27 1.27)) (hide yes))) (property "LCSC" "C11702" (at 162.56 254.00 0) (effects (font (size 1.27 1.27)) (hide yes))) (pin "1") (pin "2") (instances (project "TokenKey-RT" (path "/69bcae8e-63e2-488c-b267-fe4af22cfb6e/23672d8f-53fc-4309-8a86-d888b8c0a089" (reference "R22") (unit 1)))))
+(global_label "BOOT_MODE0_Q" (shape passive) (at 157.48 254.00 180) (fields_autoplaced yes) (effects (font (size 1.27 1.27)) (justify right)) (property "Intersheetrefs" "${INTERSHEET_REFS}" (at 157.48 254.00 0) (effects (font (size 1.27 1.27)) (hide yes))))
+(global_label "BOOT_MODE0" (shape passive) (at 167.64 254.00 0) (fields_autoplaced yes) (effects (font (size 1.27 1.27)) (justify left)) (property "Intersheetrefs" "${INTERSHEET_REFS}" (at 167.64 254.00 0) (effects (font (size 1.27 1.27)) (hide yes))))
+(text "WAKEUP (L6) and ONOFF (M6) are left unconnected and rely on their internal 100k pull-ups (IMXRT1060CEC Rev 4 Table 83: reset and default state Input, 100K PU). ONOFF also on TP5." (exclude_from_sim no) (at 30.48 22.86 0) (effects (font (size 1.27 1.27)) (justify left)))
 )
