File: hardware/schematic/usb.kicad_sch (KiCad schematic)
At the start: 5 parts, among them J1 USB-C, U6 USBLC6-2SC6

Commit message: PM review fixes: boot R_S, C51, decap note, notes, BOM fields
- MUST: add R22 (R_S) 1k 0402 0402WGF1001TCE / C11702 between Q1 drain
  (pin 3, new net BOOT_MODE0_Q) and BOOT_MODE0 (F11)
- C51 VBUS bulk 10uF 0603 -> 4.7uF 0402 (CL05A475MP5NRNC / C23733)
- docs/decisions.md: keep C11/C12; VDD_SOC total 32.5uF vs HDG ~33uF
- U3 description and root note: buck inductor is L1 (was "L2")
- mcu sheet note: WAKEUP (L6) / ONOFF (M6) rely on internal 100k PU
- APS6404L-3SQR-ZR pinout + USON-8 footprint checked vs AP Memory
  datasheet Rev 2.3 (no change); GPIO_SD_B0_04 ALT4 = FLEXSPIB_SS0_B
  confirmed in SDK fsl_iomuxc.h (H2 per DS Table 83)
- J3 TC2030 and TP1-TP5: MPN/LCSC "N/A - footprint only" + BOM_Note
- gen.py: reuse UUIDs from existing files (stable diffs), runs in-repo;
  netlist.json ignored
- kicad-cli sch erc: 0 errors, 0 warnings

Fixes #8
Parts:
- C51: value 10uF -> 4.7uF; footprint Capacitor_SMD:C_0603_1608Metric -> Capacitor_SMD:C_0402_1005Metric; LCSC C19702 -> C23733; MPN CL10A106KP8NNNC -> CL05A475MP5NRNC
Changed lines of the file:
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@@
 (global_label "USB_DN" (shape passive) (at 76.20 119.38 0) (fields_autoplaced yes) (effects (font (size 1.27 1.27)) (justify left)) (property "Intersheetrefs" "${INTERSHEET_REFS}" (at 76.20 119.38 0) (effects (font (size 1.27 1.27)) (hide yes))))
 (global_label "VBUS" (shape passive) (at 76.20 121.92 0) (fields_autoplaced yes) (effects (font (size 1.27 1.27)) (justify left)) (property "Intersheetrefs" "${INTERSHEET_REFS}" (at 76.20 121.92 0) (effects (font (size 1.27 1.27)) (hide yes))))
-(symbol (lib_id "TokenKey:C") (at 60.96 139.70 0) (unit 1) (exclude_from_sim no) (in_bom yes) (on_board yes) (dnp no) (property "Reference" "C51" (at 60.96 135.89 0) (effects (font (size 1.27 1.27)))) (property "Value" "10uF" (at 60.96 143.51 0) (effects (font (size 1.27 1.27)))) (property "Footprint" "Capacitor_SMD:C_0603_1608Metric" (at 60.96 146.05 0) (effects (font (size 1.27 1.27)) (hide yes))) (property "Datasheet" "" (at 60.96 139.70 0) (effects (font (size 1.27 1.27)) (hide yes))) (property "Description" "VBUS bulk at connector" (at 60.96 139.70 0) (effects (font (size 1.27 1.27)) (hide yes))) (property "MPN" "CL10A106KP8NNNC" (at 60.96 139.70 0) (effects (font (size 1.27 1.27)) (hide yes))) (property "LCSC" "C19702" (at 60.96 139.70 0) (effects (font (size 1.27 1.27)) (hide yes))) (pin "1") (pin "2") (instances (project "TokenKey-RT" (path "/69bcae8e-63e2-488c-b267-fe4af22cfb6e/16ce6155-0cb1-46d2-a62f-e2058aebe992" (reference "C51") (unit 1)))))
+(symbol (lib_id "TokenKey:C") (at 60.96 139.70 0) (unit 1) (exclude_from_sim no) (in_bom yes) (on_board yes) (dnp no) (property "Reference" "C51" (at 60.96 135.89 0) (effects (font (size 1.27 1.27)))) (property "Value" "4.7uF" (at 60.96 143.51 0) (effects (font (size 1.27 1.27)))) (property "Footprint" "Capacitor_SMD:C_0402_1005Metric" (at 60.96 146.05 0) (effects (font (size 1.27 1.27)) (hide yes))) (property "Datasheet" "" (at 60.96 139.70 0) (effects (font (size 1.27 1.27)) (hide yes))) (property "Description" "VBUS bulk at connector (PM review: 4.7uF)" (at 60.96 139.70 0) (effects (font (size 1.27 1.27)) (hide yes))) (property "MPN" "CL05A475MP5NRNC" (at 60.96 139.70 0) (effects (font (size 1.27 1.27)) (hide yes))) (property "LCSC" "C23733" (at 60.96 139.70 0) (effects (font (size 1.27 1.27)) (hide yes))) (pin "1") (pin "2") (instances (project "TokenKey-RT" (path "/69bcae8e-63e2-488c-b267-fe4af22cfb6e/16ce6155-0cb1-46d2-a62f-e2058aebe992" (reference "C51") (unit 1)))))
 (global_label "VBUS" (shape passive) (at 55.88 139.70 180) (fields_autoplaced yes) (effects (font (size 1.27 1.27)) (justify right)) (property "Intersheetrefs" "${INTERSHEET_REFS}" (at 55.88 139.70 0) (effects (font (size 1.27 1.27)) (hide yes))))
 (global_label "GND" (shape passive) (at 66.04 139.70 0) (fields_autoplaced yes) (effects (font (size 1.27 1.27)) (justify left)) (property "Intersheetrefs" "${INTERSHEET_REFS}" (at 66.04 139.70 0) (effects (font (size 1.27 1.27)) (hide yes))))

Commit message: BOM: second source for 4.7uF 0402 (C23733 out of stock)
- MPN_Alt CL05A475KP5NRNC / LCSC_Alt C368809 (Samsung, 4.7uF 10V X5R
  +/-10% 0402, 1,355,750 in stock at LCSC on 2026-10-19) on all 12
  4.7uF parts (C11, C12, C17, C20, C22, C25, C30, C32, C35, C39, C42, C51)
- primary CL05A475MP5NRNC / C23733 kept; out of stock at LCSC today
- kicad-cli sch erc: 0 errors, 0 warnings

Fixes #8
Parts:
- C51: LCSC_Alt (none) -> C368809; MPN_Alt (none) -> CL05A475KP5NRNC
Changed lines of the file:
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@@
 (global_label "USB_DN" (shape passive) (at 76.20 119.38 0) (fields_autoplaced yes) (effects (font (size 1.27 1.27)) (justify left)) (property "Intersheetrefs" "${INTERSHEET_REFS}" (at 76.20 119.38 0) (effects (font (size 1.27 1.27)) (hide yes))))
 (global_label "VBUS" (shape passive) (at 76.20 121.92 0) (fields_autoplaced yes) (effects (font (size 1.27 1.27)) (justify left)) (property "Intersheetrefs" "${INTERSHEET_REFS}" (at 76.20 121.92 0) (effects (font (size 1.27 1.27)) (hide yes))))
-(symbol (lib_id "TokenKey:C") (at 60.96 139.70 0) (unit 1) (exclude_from_sim no) (in_bom yes) (on_board yes) (dnp no) (property "Reference" "C51" (at 60.96 135.89 0) (effects (font (size 1.27 1.27)))) (property "Value" "4.7uF" (at 60.96 143.51 0) (effects (font (size 1.27 1.27)))) (property "Footprint" "Capacitor_SMD:C_0402_1005Metric" (at 60.96 146.05 0) (effects (font (size 1.27 1.27)) (hide yes))) (property "Datasheet" "" (at 60.96 139.70 0) (effects (font (size 1.27 1.27)) (hide yes))) (property "Description" "VBUS bulk at connector (PM review: 4.7uF)" (at 60.96 139.70 0) (effects (font (size 1.27 1.27)) (hide yes))) (property "MPN" "CL05A475MP5NRNC" (at 60.96 139.70 0) (effects (font (size 1.27 1.27)) (hide yes))) (property "LCSC" "C23733" (at 60.96 139.70 0) (effects (font (size 1.27 1.27)) (hide yes))) (pin "1") (pin "2") (instances (project "TokenKey-RT" (path "/69bcae8e-63e2-488c-b267-fe4af22cfb6e/16ce6155-0cb1-46d2-a62f-e2058aebe992" (reference "C51") (unit 1)))))
+(symbol (lib_id "TokenKey:C") (at 60.96 139.70 0) (unit 1) (exclude_from_sim no) (in_bom yes) (on_board yes) (dnp no) (property "Reference" "C51" (at 60.96 135.89 0) (effects (font (size 1.27 1.27)))) (property "Value" "4.7uF" (at 60.96 143.51 0) (effects (font (size 1.27 1.27)))) (property "Footprint" "Capacitor_SMD:C_0402_1005Metric" (at 60.96 146.05 0) (effects (font (size 1.27 1.27)) (hide yes))) (property "Datasheet" "" (at 60.96 139.70 0) (effects (font (size 1.27 1.27)) (hide yes))) (property "Description" "VBUS bulk at connector (PM review: 4.7uF)" (at 60.96 139.70 0) (effects (font (size 1.27 1.27)) (hide yes))) (property "MPN" "CL05A475MP5NRNC" (at 60.96 139.70 0) (effects (font (size 1.27 1.27)) (hide yes))) (property "LCSC" "C23733" (at 60.96 139.70 0) (effects (font (size 1.27 1.27)) (hide yes))) (property "MPN_Alt" "CL05A475KP5NRNC" (at 60.96 139.70 0) (effects (font (size 1.27 1.27)) (hide yes))) (property "LCSC_Alt" "C368809" (at 60.96 139.70 0) (effects (font (size 1.27 1.27)) (hide yes))) (pin "1") (pin "2") (instances (project "TokenKey-RT" (path "/69bcae8e-63e2-488c-b267-fe4af22cfb6e/16ce6155-0cb1-46d2-a62f-e2058aebe992" (reference "C51") (unit 1)))))
 (global_label "VBUS" (shape passive) (at 55.88 139.70 180) (fields_autoplaced yes) (effects (font (size 1.27 1.27)) (justify right)) (property "Intersheetrefs" "${INTERSHEET_REFS}" (at 55.88 139.70 0) (effects (font (size 1.27 1.27)) (hide yes))))
 (global_label "GND" (shape passive) (at 66.04 139.70 0) (fields_autoplaced yes) (effects (font (size 1.27 1.27)) (justify left)) (property "Intersheetrefs" "${INTERSHEET_REFS}" (at 66.04 139.70 0) (effects (font (size 1.27 1.27)) (hide yes))))
