File: hardware/schematic/power.kicad_sch (KiCad schematic)
At the start: 50 parts, among them U2 AP2112K-3.3TRG1, U3 TLV62569DBVR

Commit message: Schematic baseline: BGA land pattern, OLED module, 220nF second source
- U1 footprint: per NXP SOT1546-2 / case outline 98ASA01088D Rev O
  (IMXRT1060CEC Rev 4 Fig. 53; balls d0.25-0.35) and NXP AN4982 Rev 4
  s4.2: 0.325 mm NSMD Cu pads, 0.450 mm mask opening (was 0.30 mm guess)
- J2 OLED: HS HS96L03W2C03, LCSC C5248080 (SSD1315, SSD1306-compatible);
  pins 1 GND 2 VCC 3 SCL 4 SDA per datasheet V1.0 (matches existing
  nets); 3.3 V max, no onboard LDO, external pull-ups R14/R15 kept;
  27.3x27.8 mm, 4x d2.5 holes on 23.3x23.8 mm
- 220nF 0402: add MPN_Alt CL05B224KO5NNNC / LCSC_Alt C16772 (16V X7R)
  as second source to C47129 on all 14 parts
- docs/pin-map.md and generators updated to match
- kicad-cli sch erc: 0 errors, 0 warnings

Fixes #8
Parts:
- C10, C14, C15, C16, C19, C21, C23, C24, C27, C43, C6, C7, C8, C9: LCSC_Alt (none) -> C16772; MPN_Alt (none) -> CL05B224KO5NNNC

Commit message: BOM: second source for 4.7uF 0402 (C23733 out of stock)
- MPN_Alt CL05A475KP5NRNC / LCSC_Alt C368809 (Samsung, 4.7uF 10V X5R
  +/-10% 0402, 1,355,750 in stock at LCSC on 2026-10-19) on all 12
  4.7uF parts (C11, C12, C17, C20, C22, C25, C30, C32, C35, C39, C42, C51)
- primary CL05A475MP5NRNC / C23733 kept; out of stock at LCSC today
- kicad-cli sch erc: 0 errors, 0 warnings

Fixes #8
Parts:
- C11, C12, C17, C20, C22, C25, C30, C32, C35, C39, C42: LCSC_Alt (none) -> C368809; MPN_Alt (none) -> CL05A475KP5NRNC

Commit message: L2: low-profile 4.7uH DCDC inductor (TDK VLS3015CX-4R7M-1, alt SWPA3015S4R7MT) + OLED mechanical data
- L2 (power.kicad_sch, via KiCad MCP edit_schematic_component): VLS3015CX-4R7M-1 / C3220938,
  3.0x3.0x1.5 mm max, DCR 0.137R max, Isat 1.37A; MPN_Alt SWPA3015S4R7MT / LCSC_Alt C19398.
- New footprint TokenKey:L_3.0x3.0mm_TDK_VLS3015CX (TDK land: 2x 1.0x3.0 mm pads, +/-1.0 mm),
  created with the MCP create_footprint tool.
- docs/decisions.md: L2 rationale + HS96L03W2C03 mechanical offsets.
- pin-map note updated. run_erc: 0 violations.

Fixes #24
Parts:
- L2: footprint Inductor_SMD:L_Sunlord_SWPA4020S -> TokenKey:L_3.0x3.0mm_TDK_VLS3015CX; BOM_Note (none) -> Alt Sunlord SWPA3015S4R7MT (3.0x3.0x1.5, DCR 0.163R max, Is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; LCSC C48427 -> C3220938; LCSC_Alt (none) -> C19398; MPN SWPA4020S4R7MT -> VLS3015CX-4R7M-1; MPN_Alt (none) -> SWPA3015S4R7MT; Manufacturer (none) -> TDK
Changed lines of the file:
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@@
 (global_label "3V3" (shape passive) (at 55.88 243.84 180) (fields_autoplaced yes) (effects (font (size 1.27 1.27)) (justify right)) (property "Intersheetrefs" "${INTERSHEET_REFS}" (at 55.88 243.84 0) (effects (font (size 1.27 1.27)) (hide yes))))
 (global_label "GND" (shape passive) (at 66.04 243.84 0) (fields_autoplaced yes) (effects (font (size 1.27 1.27)) (justify left)) (property "Intersheetrefs" "${INTERSHEET_REFS}" (at 66.04 243.84 0) (effects (font (size 1.27 1.27)) (hide yes))))
-(symbol (lib_id "TokenKey:L") (at 60.96 261.62 0) (unit 1) (exclude_from_sim no) (in_bom yes) (on_board yes) (dnp no) (property "Reference" "L2" (at 60.96 257.81 0) (effects (font (size 1.27 1.27)))) (property "Value" "4.7uH" (at 60.96 265.43 0) (effects (font (size 1.27 1.27)))) (property "Footprint" "Inductor_SMD:L_Sunlord_SWPA4020S" (at 60.96 267.97 0) (effects (font (size 1.27 1.27)) (hide yes))) (property "Datasheet" "" (at 60.96 261.62 0) (effects (font (size 1.27 1.27)) (hide yes))) (property "Description" "RT1062 DCDC inductor (HDG: 4.7-10uH, Isat>1A, DCR<0.2R)" (at 60.96 261.62 0) (effects (font (size 1.27 1.27)) (hide yes))) (property "MPN" "SWPA4020S4R7MT" (at 60.96 261.62 0) (effects (font (size 1.27 1.27)) (hide yes))) (property "LCSC" "C48427" (at 60.96 261.62 0) (effects (font (size 1.27 1.27)) (hide yes))) (pin "1") (pin "2") (instances (project "TokenKey-RT" (path "/69bcae8e-63e2-488c-b267-fe4af22cfb6e/ac6a820c-90cd-4dc7-a10d-64e8a5622379" (reference "L2") (unit 1)))))
+(symbol (lib_id "TokenKey:L") (at 60.96 261.62 0) (unit 1) (exclude_from_sim no) (in_bom yes) (on_board yes) (dnp no) (property "Reference" "L2" (at 60.96 257.81 0) (effects (font (size 1.27 1.27)))) (property "Value" "4.7uH" (at 60.96 265.43 0) (effects (font (size 1.27 1.27)))) (property "Footprint" "TokenKey:L_3.0x3.0mm_TDK_VLS3015CX" (at 60.96 267.97 0) (effects (font (size 1.27 1.27)) (hide yes))) (property "Datasheet" "" (at 60.96 261.62 0) (effects (font (size 1.27 1.27)) (hide yes))) (property "Description" "RT1062 DCDC inductor 4.7uH 20%, 3.0x3.0x1.5mm max, DCR 0.137R max, Isat 1.37A (HDG: 4.7-10uH, Isat>1A, DCR<0.2R)" (at 60.96 261.62 0) (effects (font (size 1.27 1.27)) (hide yes))) (property "MPN" "VLS3015CX-4R7M-1" (at 60.96 261.62 0) (effects (font (size 1.27 1.27)) (hide yes))) (property "LCSC" "C3220938" (at 60.96 261.62 0) (effects (font (size 1.27 1.27)) (hide yes)))
+    (property "Manufacturer" "TDK" (at 60.96 261.62 0)
+      (effects (font (size 1.27 1.27)) (hide yes))
+    )
+    (property "MPN_Alt" "SWPA3015S4R7MT" (at 60.96 261.62 0)
+      (effects (font (size 1.27 1.27)) (hide yes))
+    )
+    (property "LCSC_Alt" "C19398" (at 60.96 261.62 0)
+      (effects (font (size 1.27 1.27)) (hide yes))
+    )
+    (property "BOM_Note" "Alt Sunlord SWPA3015S4R7MT (3.0x3.0x1.5, DCR 0.163R max, Isat 1.10A) fits same land; JLC Extended" (at 60.96 261.62 0)
+      (effects (font (size 1.27 1.27)) (hide yes))
+    ) (pin "1") (pin "2") (instances (project "TokenKey-RT" (path "/69bcae8e-63e2-488c-b267-fe4af22cfb6e/ac6a820c-90cd-4dc7-a10d-64e8a5622379" (reference "L2") (unit 1)))))
 (global_label "DCDC_LP" (shape passive) (at 55.88 261.62 180) (fields_autoplaced yes) (effects (font (size 1.27 1.27)) (justify right)) (property "Intersheetrefs" "${INTERSHEET_REFS}" (at 55.88 261.62 0) (effects (font (size 1.27 1.27)) (hide yes))))
 (global_label "VDD_SOC" (shape passive) (at 66.04 261.62 0) (fields_autoplaced yes) (effects (font (size 1.27 1.27)) (justify left)) (property "Intersheetrefs" "${INTERSHEET_REFS}" (at 66.04 261.62 0) (effects (font (size 1.27 1.27)) (hide yes))))
