File: hardware/schematic/debug.kicad_sch (KiCad schematic)
At the start: 6 parts, among them J3 TC2030-NL

Commit message: PM review fixes: boot R_S, C51, decap note, notes, BOM fields
- MUST: add R22 (R_S) 1k 0402 0402WGF1001TCE / C11702 between Q1 drain
  (pin 3, new net BOOT_MODE0_Q) and BOOT_MODE0 (F11)
- C51 VBUS bulk 10uF 0603 -> 4.7uF 0402 (CL05A475MP5NRNC / C23733)
- docs/decisions.md: keep C11/C12; VDD_SOC total 32.5uF vs HDG ~33uF
- U3 description and root note: buck inductor is L1 (was "L2")
- mcu sheet note: WAKEUP (L6) / ONOFF (M6) rely on internal 100k PU
- APS6404L-3SQR-ZR pinout + USON-8 footprint checked vs AP Memory
  datasheet Rev 2.3 (no change); GPIO_SD_B0_04 ALT4 = FLEXSPIB_SS0_B
  confirmed in SDK fsl_iomuxc.h (H2 per DS Table 83)
- J3 TC2030 and TP1-TP5: MPN/LCSC "N/A - footprint only" + BOM_Note
- gen.py: reuse UUIDs from existing files (stable diffs), runs in-repo;
  netlist.json ignored
- kicad-cli sch erc: 0 errors, 0 warnings

Fixes #8
Parts:
- J3: BOM_Note (none) -> Footprint only - nothing to buy (no component placed; exclu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; LCSC N/A -> N/A - footprint only; MPN TC2030-NL (footprint only) -> N/A - footprint only
- TP1, TP2, TP3, TP4, TP5: BOM_Note (none) -> Footprint only - nothing to buy (no component placed; exclu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; LCSC N/A -> N/A - footprint only; MPN Test pad (no part) -> N/A - footprint only

Commit message: BOM: exclude J3 (TC2030) and TP1-TP5 from BOM (in_bom no)
Scripted hand edit of hardware/schematic/debug.kicad_sch (PM-approved
exception): the KiCad MCP connector has no tool for the symbol in_bom
attribute. A Python script changed (in_bom yes) -> (in_bom no) on the
J3 and TP1-TP5 symbol lines only; git diff = 6 lines, in_bom token only.
run_erc (user-kicad): 0 violations. export_sch_bom confirms the six refs
are absent from the BOM.

Fixes #32
Parts:
- J3, TP1, TP2, TP3, TP4, TP5: now left out of the parts list
