File: hardware/schematic/ui.kicad_sch (KiCad schematic)
At the start: 15 parts, among them J2 SSD1306 OLED 128x64, SW2 EC11E18244A5, SW3 BTN1, SW4 BTN2

Commit message: Schematic baseline: BGA land pattern, OLED module, 220nF second source
- U1 footprint: per NXP SOT1546-2 / case outline 98ASA01088D Rev O
  (IMXRT1060CEC Rev 4 Fig. 53; balls d0.25-0.35) and NXP AN4982 Rev 4
  s4.2: 0.325 mm NSMD Cu pads, 0.450 mm mask opening (was 0.30 mm guess)
- J2 OLED: HS HS96L03W2C03, LCSC C5248080 (SSD1315, SSD1306-compatible);
  pins 1 GND 2 VCC 3 SCL 4 SDA per datasheet V1.0 (matches existing
  nets); 3.3 V max, no onboard LDO, external pull-ups R14/R15 kept;
  27.3x27.8 mm, 4x d2.5 holes on 23.3x23.8 mm
- 220nF 0402: add MPN_Alt CL05B224KO5NNNC / LCSC_Alt C16772 (16V X7R)
  as second source to C47129 on all 14 parts
- docs/pin-map.md and generators updated to match
- kicad-cli sch erc: 0 errors, 0 warnings

Fixes #8
Parts:
- J2: value SSD1306 OLED 128x64 -> OLED 0.96in 128x64 I2C (SSD1315); LCSC UNVERIFIED -> C5248080; MPN SSD1306 0.96in I2C module (generic) -> HS96L03W2C03
Changed lines of the file:
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@@
 (kicad_sch (version 20250114) (generator "eeschema") (generator_version "9.0") (paper "A3") (title_block (title "UI: OLED, encoder, buttons, LED") (company "TokenKey RT") (rev "A0-draft") (comment 1 "Generated by tools/gen.py - frozen baseline pin map"))
-(symbol (lib_id "TokenKey:OLED_I2C_4P") (at 66.04 38.10 0) (unit 1) (exclude_from_sim no) (in_bom yes) (on_board yes) (dnp no) (property "Reference" "J2" (at 66.04 34.29 0) (effects (font (size 1.27 1.27)))) (property "Value" "SSD1306 OLED 128x64" (at 66.04 44.45 0) (effects (font (size 1.27 1.27)))) (property "Footprint" "Connector_PinHeader_2.54mm:PinHeader_1x04_P2.54mm_Vertical" (at 66.04 46.99 0) (effects (font (size 1.27 1.27)) (hide yes))) (property "Datasheet" "" (at 66.04 38.10 0) (effects (font (size 1.27 1.27)) (hide yes))) (property "Description" "Module pin order GND/VCC/SCL/SDA UNVERIFIED - check chosen module" (at 66.04 38.10 0) (effects (font (size 1.27 1.27)) (hide yes))) (property "MPN" "SSD1306 0.96in I2C module (generic)" (at 66.04 38.10 0) (effects (font (size 1.27 1.27)) (hide yes))) (property "LCSC" "UNVERIFIED" (at 66.04 38.10 0) (effects (font (size 1.27 1.27)) (hide yes))) (pin "1") (pin "2") (pin "3") (pin "4") (instances (project "TokenKey-RT" (path "/69bcae8e-63e2-488c-b267-fe4af22cfb6e/912f45be-b651-4781-b3b5-bccddac83cec" (reference "J2") (unit 1)))))
+(symbol (lib_id "TokenKey:OLED_I2C_4P") (at 66.04 38.10 0) (unit 1) (exclude_from_sim no) (in_bom yes) (on_board yes) (dnp no) (property "Reference" "J2" (at 66.04 34.29 0) (effects (font (size 1.27 1.27)))) (property "Value" "OLED 0.96in 128x64 I2C (SSD1315)" (at 66.04 44.45 0) (effects (font (size 1.27 1.27)))) (property "Footprint" "Connector_PinHeader_2.54mm:PinHeader_1x04_P2.54mm_Vertical" (at 66.04 46.99 0) (effects (font (size 1.27 1.27)) (hide yes))) (property "Datasheet" "" (at 66.04 38.10 0) (effects (font (size 1.27 1.27)) (hide yes))) (property "Description" "HS HS96L03W2C03 module (datasheet V1.0 s1.4/1.5): pins 1 GND 2 VCC 3 SCL 4 SDA, 2.54 mm; VCC 2.8-3.3 V max (no on-module LDO, 3V3 only); needs external SCL/SDA pull-ups (R14/R15); PCB 27.3x27.8 mm, 4x d2.5 mm holes on 23.3x23.8 mm. SSD1315 = SSD1306-compatible. Alt (out of stock): Jixin JX040102-1 C284855, SSD1306 + LDO, 30x29 mm, different hole pattern" (at 66.04 38.10 0) (effects (font (size 1.27 1.27)) (hide yes))) (property "MPN" "HS96L03W2C03" (at 66.04 38.10 0) (effects (font (size 1.27 1.27)) (hide yes))) (property "LCSC" "C5248080" (at 66.04 38.10 0) (effects (font (size 1.27 1.27)) (hide yes))) (pin "1") (pin "2") (pin "3") (pin "4") (instances (project "TokenKey-RT" (path "/69bcae8e-63e2-488c-b267-fe4af22cfb6e/912f45be-b651-4781-b3b5-bccddac83cec" (reference "J2") (unit 1)))))
 (global_label "GND" (shape passive) (at 55.88 38.10 180) (fields_autoplaced yes) (effects (font (size 1.27 1.27)) (justify right)) (property "Intersheetrefs" "${INTERSHEET_REFS}" (at 55.88 38.10 0) (effects (font (size 1.27 1.27)) (hide yes))))
 (global_label "3V3" (shape passive) (at 55.88 40.64 180) (fields_autoplaced yes) (effects (font (size 1.27 1.27)) (justify right)) (property "Intersheetrefs" "${INTERSHEET_REFS}" (at 55.88 40.64 0) (effects (font (size 1.27 1.27)) (hide yes))))

Commit message: J2: low-profile 1x4 2.54 mm socket, 3.0 mm insulator (XFCN MF254V-11-04-0743)
Via KiCad MCP edit_schematic_component on ui.kicad_sch:
- MPN MF254V-11-04-0743 / LCSC C2889986 (XFCN), insulator 3.00+/-0.10 mm
  per XFCN drawing MF254V-11-xx-0743 (2020-04-12).
- Alt XDM254C-1-04-Z-3.0-G0 / C19184298 (chxunda).
- Footprint Connector_PinSocket_2.54mm:PinSocket_1x04_P2.54mm_Vertical
  (same pad pattern as before: pin 1 at origin, pitch 2.54 along +y).
- OLED module kept as Module_MPN/Module_LCSC; BOM_Note: round machined
  pins required on the OLED side.
run_erc: 0 violations.

Fixes #36
Parts:
- J2: value OLED 0.96in 128x64 I2C (SSD1315) -> Socket 1x04 P2.54 H3.0 (OLED); footprint Connector_PinHeader_2.54mm:PinHeader_1x04_P2.54mm_Vertical -> Connector_PinSocket_2.54mm:PinSocket_1x04_P2.54mm_Vertical; BOM_Note (none) -> Machined round-hole socket, insulator 3.00+/-0.10 mm (XFCN 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; LCSC C5248080 -> C2889986; LCSC_Alt (none) -> C19184298; MPN HS96L03W2C03 -> MF254V-11-04-0743; MPN_Alt (none) -> XDM254C-1-04-Z-3.0-G0; Manufacturer (none) -> XFCN; Module_LCSC (none) -> C5248080; Module_MPN (none) -> HS96L03W2C03
Changed lines of the file:
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@@
 (kicad_sch (version 20250114) (generator "eeschema") (generator_version "9.0") (paper "A3") (title_block (title "UI: OLED, encoder, buttons, LED") (company "TokenKey RT") (rev "A0-draft") (comment 1 "Generated by tools/gen.py - frozen baseline pin map"))
-(symbol (lib_id "TokenKey:OLED_I2C_4P") (at 66.04 38.10 0) (unit 1) (exclude_from_sim no) (in_bom yes) (on_board yes) (dnp no) (property "Reference" "J2" (at 66.04 34.29 0) (effects (font (size 1.27 1.27)))) (property "Value" "OLED 0.96in 128x64 I2C (SSD1315)" (at 66.04 44.45 0) (effects (font (size 1.27 1.27)))) (property "Footprint" "Connector_PinHeader_2.54mm:PinHeader_1x04_P2.54mm_Vertical" (at 66.04 46.99 0) (effects (font (size 1.27 1.27)) (hide yes))) (property "Datasheet" "" (at 66.04 38.10 0) (effects (font (size 1.27 1.27)) (hide yes))) (property "Description" "HS HS96L03W2C03 module (datasheet V1.0 s1.4/1.5): pins 1 GND 2 VCC 3 SCL 4 SDA, 2.54 mm; VCC 2.8-3.3 V max (no on-module LDO, 3V3 only); needs external SCL/SDA pull-ups (R14/R15); PCB 27.3x27.8 mm, 4x d2.5 mm holes on 23.3x23.8 mm. SSD1315 = SSD1306-compatible. Alt (out of stock): Jixin JX040102-1 C284855, SSD1306 + LDO, 30x29 mm, different hole pattern" (at 66.04 38.10 0) (effects (font (size 1.27 1.27)) (hide yes))) (property "MPN" "HS96L03W2C03" (at 66.04 38.10 0) (effects (font (size 1.27 1.27)) (hide yes))) (property "LCSC" "C5248080" (at 66.04 38.10 0) (effects (font (size 1.27 1.27)) (hide yes))) (pin "1") (pin "2") (pin "3") (pin "4") (instances (project "TokenKey-RT" (path "/69bcae8e-63e2-488c-b267-fe4af22cfb6e/912f45be-b651-4781-b3b5-bccddac83cec" (reference "J2") (unit 1)))))
+(symbol (lib_id "TokenKey:OLED_I2C_4P") (at 66.04 38.10 0) (unit 1) (exclude_from_sim no) (in_bom yes) (on_board yes) (dnp no) (property "Reference" "J2" (at 66.04 34.29 0) (effects (font (size 1.27 1.27)))) (property "Value" "Socket 1x04 P2.54 H3.0 (OLED)" (at 66.04 44.45 0) (effects (font (size 1.27 1.27)))) (property "Footprint" "Connector_PinSocket_2.54mm:PinSocket_1x04_P2.54mm_Vertical" (at 66.04 46.99 0) (effects (font (size 1.27 1.27)) (hide yes))) (property "Datasheet" "" (at 66.04 38.10 0) (effects (font (size 1.27 1.27)) (hide yes))) (property "Description" "HS HS96L03W2C03 module (datasheet V1.0 s1.4/1.5): pins 1 GND 2 VCC 3 SCL 4 SDA, 2.54 mm; VCC 2.8-3.3 V max (no on-module LDO, 3V3 only); needs external SCL/SDA pull-ups (R14/R15); PCB 27.3x27.8 mm, 4x d2.5 mm holes on 23.3x23.8 mm. SSD1315 = SSD1306-compatible. Alt (out of stock): Jixin JX040102-1 C284855, SSD1306 + LDO, 30x29 mm, different hole pattern" (at 66.04 38.10 0) (effects (font (size 1.27 1.27)) (hide yes))) (property "MPN" "MF254V-11-04-0743" (at 66.04 38.10 0) (effects (font (size 1.27 1.27)) (hide yes))) (property "LCSC" "C2889986" (at 66.04 38.10 0) (effects (font (size 1.27 1.27)) (hide yes)))
+    (property "Manufacturer" "XFCN" (at 66.04 38.1 0)
+      (effects (font (size 1.27 1.27)) (hide yes))
+    )
+    (property "MPN_Alt" "XDM254C-1-04-Z-3.0-G0" (at 66.04 38.1 0)
+      (effects (font (size 1.27 1.27)) (hide yes))
+    )
+    (property "LCSC_Alt" "C19184298" (at 66.04 38.1 0)
+      (effects (font (size 1.27 1.27)) (hide yes))
+    )
+    (property "Module_MPN" "HS96L03W2C03" (at 66.04 38.1 0)
+      (effects (font (size 1.27 1.27)) (hide yes))
+    )
+    (property "Module_LCSC" "C5248080" (at 66.04 38.1 0)
+      (effects (font (size 1.27 1.27)) (hide yes))
+    )
+    (property "BOM_Note" "Machined round-hole socket, insulator 3.00+/-0.10 mm (XFCN dwg MF254V-11-xx-0743, 2020-04-12); accepts round pins only (rated with d0.432 test pin; alt accepts d0.40-0.60) - OLED needs a round machined-pin male header, standard 0.64 mm square pins will not fit. OLED module HS96L03W2C03/C5248080 ordered separately (Module_MPN/Module_LCSC)." (at 66.04 38.1 0)
+      (effects (font (size 1.27 1.27)) (hide yes))
+    ) (pin "1") (pin "2") (pin "3") (pin "4") (instances (project "TokenKey-RT" (path "/69bcae8e-63e2-488c-b267-fe4af22cfb6e/912f45be-b651-4781-b3b5-bccddac83cec" (reference "J2") (unit 1)))))
 (global_label "GND" (shape passive) (at 55.88 38.10 180) (fields_autoplaced yes) (effects (font (size 1.27 1.27)) (justify right)) (property "Intersheetrefs" "${INTERSHEET_REFS}" (at 55.88 38.10 0) (effects (font (size 1.27 1.27)) (hide yes))))
 (global_label "3V3" (shape passive) (at 55.88 40.64 180) (fields_autoplaced yes) (effects (font (size 1.27 1.27)) (justify right)) (property "Intersheetrefs" "${INTERSHEET_REFS}" (at 55.88 40.64 0) (effects (font (size 1.27 1.27)) (hide yes))))

Commit message: J2/OLED: round machined-pin male header HCTL PZ254-1-04-Z-C (C5156431)
- J2 (ui.kicad_sch) via user-kicad edit_schematic_component: added
  Module_Header_MPN PZ254-1-04-Z-C, Module_Header_LCSC C5156431,
  Module_Header_Manufacturer HCTL, Module_Header_MPN_Alt TS-104-G-AA,
  Module_Header_LCSC_Alt C3331270; updated BOM_Note.
- ui sheet assembly note via add_schematic_text at (25.4, 25.4): stock
  square header removed, replaced with the round-pin header; nominal
  stack 3.00 + 3.00 + 2.65 = 8.65 mm above board top.
- docs/decisions.md row.
run_erc: 0 violations.

Fixes #44
Parts:
- J2: BOM_Note Machined round-hole socket, insulator 3.00+/-0.10 mm (XFCN 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 -> J2 = XFCN MF254V-11-04-0743 machined round-hole socket, ins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; Module_Header_LCSC (none) -> C5156431; Module_Header_LCSC_Alt (none) -> C3331270; Module_Header_MPN (none) -> PZ254-1-04-Z-C; Module_Header_MPN_Alt (none) -> TS-104-G-AA; Module_Header_Manufacturer (none) -> HCTL
Other:
- note added: "ASSEMBLY (J2/OLED): remove the OLED module's stock square-pin header and replace it with round machined-pin header HCTL PZ254-1-04-Z-C (LCSC C5156431), d0.50 mm mating end into J2 socket, d0.60 mm end soldered through the OLED PCB. Stack above board top (nominal): socket 3.00 + header plastic 3.00 + OLED module 2.65 = 8.65 mm."
Changed lines of the file:
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@@
       (effects (font (size 1.27 1.27)) (hide yes))
     )
-    (property "BOM_Note" "Machined round-hole socket, insulator 3.00+/-0.10 mm (XFCN dwg MF254V-11-xx-0743, 2020-04-12); accepts round pins only (rated with d0.432 test pin; alt accepts d0.40-0.60) - OLED needs a round machined-pin male header, standard 0.64 mm square pins will not fit. OLED module HS96L03W2C03/C5248080 ordered separately (Module_MPN/Module_LCSC)." (at 66.04 38.1 0)
+    (property "BOM_Note" "J2 = XFCN MF254V-11-04-0743 machined round-hole socket, insulator 3.00+/-0.10 mm (dwg MF254V-11-xx-0743, 2020-04-12); round pins only. OLED module HS96L03W2C03/C5248080 ordered separately (Module_MPN/Module_LCSC). Remove the module's stock square header; fit HCTL PZ254-1-04-Z-C/C5156431 round machined-pin header (Module_Header_*): mating pin d0.50+/-0.03 x 4.13 into J2, solder tail d0.60+/-0.03 through OLED PCB, plastic 3.0 mm (dwg PZ254-1-N-Z-XX-C rev A). Alt Samtec TS-104-G-AA/C3331270 (d0.46 both ends, low stock, insulator height not confirmed). Nominal stack above board top 3.00+3.00+2.65 = 8.65 mm." (at 66.04 38.1 0)
+      (effects (font (size 1.27 1.27)) (hide yes))
+    )
+    (property "Module_Header_MPN" "PZ254-1-04-Z-C" (at 66.04 38.1 0)
+      (effects (font (size 1.27 1.27)) (hide yes))
+    )
+    (property "Module_Header_LCSC" "C5156431" (at 66.04 38.1 0)
+      (effects (font (size 1.27 1.27)) (hide yes))
+    )
+    (property "Module_Header_Manufacturer" "HCTL" (at 66.04 38.1 0)
+      (effects (font (size 1.27 1.27)) (hide yes))
+    )
+    (property "Module_Header_MPN_Alt" "TS-104-G-AA" (at 66.04 38.1 0)
+      (effects (font (size 1.27 1.27)) (hide yes))
+    )
+    (property "Module_Header_LCSC_Alt" "C3331270" (at 66.04 38.1 0)
       (effects (font (size 1.27 1.27)) (hide yes))
     ) (pin "1") (pin "2") (pin "3") (pin "4") (instances (project "TokenKey-RT" (path "/69bcae8e-63e2-488c-b267-fe4af22cfb6e/912f45be-b651-4781-b3b5-bccddac83cec" (reference "J2") (unit 1)))))
@@
 (global_label "LED_A" (shape passive) (at 132.08 73.66 180) (fields_autoplaced yes) (effects (font (size 1.27 1.27)) (justify right)) (property "Intersheetrefs" "${INTERSHEET_REFS}" (at 132.08 73.66 0) (effects (font (size 1.27 1.27)) (hide yes))))
 (global_label "GND" (shape passive) (at 147.32 73.66 0) (fields_autoplaced yes) (effects (font (size 1.27 1.27)) (justify left)) (property "Intersheetrefs" "${INTERSHEET_REFS}" (at 147.32 73.66 0) (effects (font (size 1.27 1.27)) (hide yes))))
+	(text "ASSEMBLY (J2/OLED): remove the OLED module's stock square-pin header and replace it with round machined-pin header HCTL PZ254-1-04-Z-C (LCSC C5156431),\nd0.50 mm mating end into J2 socket, d0.60 mm end soldered through the OLED PCB.\nStack above board top (nominal): socket 3.00 + header plastic 3.00 + OLED module 2.65 = 8.65 mm."
+		(exclude_from_sim no)
+		(at 25.4 25.4 0)
+		(effects
+			(font
+				(size 1.27 1.27)
+			)
+			(justify left bottom)
+		)
+	)
 )

Commit message: J2/OLED re-scope: no socket, module soldered directly to 3.0 mm header
- J2 (ui.kicad_sch) via user-kicad edit_schematic_component: Value
  "Header 1x04 P2.54 H3.0 (OLED)", footprint
  Connector_PinHeader_2.54mm:PinHeader_1x04_P2.54mm_Vertical, MPN
  PZ254-1-04-Z-C, LCSC C5156431, Manufacturer HCTL, BOM_Note updated.
  Removed MF254V socket alt fields (MPN_Alt, LCSC_Alt) and all
  Module_Header_* fields. Module_MPN/Module_LCSC kept (HS96L03W2C03 /
  C5248080, own BOM line).
- No square-pin 1x4 2.54 mm header with 3.0 mm plastic found at
  LCSC/JLC (all 2.5 mm), so PZ254-1-04-Z-C used per PM fallback.
- HAND EDIT (scripted): replaced the string of the existing ui-sheet
  assembly note (user-kicad has no text edit/delete tool). Position,
  size and uuid unchanged.
- docs/decisions.md: #44 row rewritten (single stack record:
  underside 3.0, OLED top ~5.65, envelope ~6.65 mm); #31 row: socket-era
  6.6 / 8.2 mm stack removed, points to #44 row.
run_erc: 0 violations.

Fixes #44
Parts:
- J2: value Socket 1x04 P2.54 H3.0 (OLED) -> Header 1x04 P2.54 H3.0 (OLED); footprint Connector_PinSocket_2.54mm:PinSocket_1x04_P2.54mm_Vertical -> Connector_PinHeader_2.54mm:PinHeader_1x04_P2.54mm_Vertical; BOM_Note J2 = XFCN MF254V-11-04-0743 machined round-hole socket, ins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 -> 1x4 2.54 mm male header, plastic 3.0 mm (HCTL dwg PZ254-1-N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; LCSC C2889986 -> C5156431; LCSC_Alt C19184298 -> (none); MPN MF254V-11-04-0743 -> PZ254-1-04-Z-C; MPN_Alt XDM254C-1-04-Z-3.0-G0 -> (none); Manufacturer XFCN -> HCTL; Module_Header_LCSC C5156431 -> (none); Module_Header_LCSC_Alt C3331270 -> (none); Module_Header_MPN PZ254-1-04-Z-C -> (none); Module_Header_MPN_Alt TS-104-G-AA -> (none); Module_Header_Manufacturer HCTL -> (none)
Other:
- note added: "ASSEMBLY (J2/OLED): OLED module soldered directly via 3.0 mm header (J2, HCTL PZ254-1-04-Z-C, LCSC C5156431); module stock header not used. Module underside 3.0 mm above PCB; OLED top ~5.65 mm (3.0 + 2.65); envelope ~6.65 mm with the 1.0 mm back-side feature."
- note removed: "ASSEMBLY (J2/OLED): remove the OLED module's stock square-pin header and replace it with round machined-pin header HCTL PZ254-1-04-Z-C (LCSC C5156431), d0.50 mm mating end into J2 socket, d0.60 mm end soldered through the OLED PCB. Stack above board top (nominal): socket 3.00 + header plastic 3.00 + OLED module 2.65 = 8.65 mm."
Changed lines of the file:
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@@
 (kicad_sch (version 20250114) (generator "eeschema") (generator_version "9.0") (paper "A3") (title_block (title "UI: OLED, encoder, buttons, LED") (company "TokenKey RT") (rev "A0-draft") (comment 1 "Generated by tools/gen.py - frozen baseline pin map"))
-(symbol (lib_id "TokenKey:OLED_I2C_4P") (at 66.04 38.10 0) (unit 1) (exclude_from_sim no) (in_bom yes) (on_board yes) (dnp no) (property "Reference" "J2" (at 66.04 34.29 0) (effects (font (size 1.27 1.27)))) (property "Value" "Socket 1x04 P2.54 H3.0 (OLED)" (at 66.04 44.45 0) (effects (font (size 1.27 1.27)))) (property "Footprint" "Connector_PinSocket_2.54mm:PinSocket_1x04_P2.54mm_Vertical" (at 66.04 46.99 0) (effects (font (size 1.27 1.27)) (hide yes))) (property "Datasheet" "" (at 66.04 38.10 0) (effects (font (size 1.27 1.27)) (hide yes))) (property "Description" "HS HS96L03W2C03 module (datasheet V1.0 s1.4/1.5): pins 1 GND 2 VCC 3 SCL 4 SDA, 2.54 mm; VCC 2.8-3.3 V max (no on-module LDO, 3V3 only); needs external SCL/SDA pull-ups (R14/R15); PCB 27.3x27.8 mm, 4x d2.5 mm holes on 23.3x23.8 mm. SSD1315 = SSD1306-compatible. Alt (out of stock): Jixin JX040102-1 C284855, SSD1306 + LDO, 30x29 mm, different hole pattern" (at 66.04 38.10 0) (effects (font (size 1.27 1.27)) (hide yes))) (property "MPN" "MF254V-11-04-0743" (at 66.04 38.10 0) (effects (font (size 1.27 1.27)) (hide yes))) (property "LCSC" "C2889986" (at 66.04 38.10 0) (effects (font (size 1.27 1.27)) (hide yes)))
-    (property "Manufacturer" "XFCN" (at 66.04 38.1 0)
-      (effects (font (size 1.27 1.27)) (hide yes))
-    )
-    (property "MPN_Alt" "XDM254C-1-04-Z-3.0-G0" (at 66.04 38.1 0)
-      (effects (font (size 1.27 1.27)) (hide yes))
-    )
-    (property "LCSC_Alt" "C19184298" (at 66.04 38.1 0)
+(symbol (lib_id "TokenKey:OLED_I2C_4P") (at 66.04 38.10 0) (unit 1) (exclude_from_sim no) (in_bom yes) (on_board yes) (dnp no) (property "Reference" "J2" (at 66.04 34.29 0) (effects (font (size 1.27 1.27)))) (property "Value" "Header 1x04 P2.54 H3.0 (OLED)" (at 66.04 44.45 0) (effects (font (size 1.27 1.27)))) (property "Footprint" "Connector_PinHeader_2.54mm:PinHeader_1x04_P2.54mm_Vertical" (at 66.04 46.99 0) (effects (font (size 1.27 1.27)) (hide yes))) (property "Datasheet" "" (at 66.04 38.10 0) (effects (font (size 1.27 1.27)) (hide yes))) (property "Description" "HS HS96L03W2C03 module (datasheet V1.0 s1.4/1.5): pins 1 GND 2 VCC 3 SCL 4 SDA, 2.54 mm; VCC 2.8-3.3 V max (no on-module LDO, 3V3 only); needs external SCL/SDA pull-ups (R14/R15); PCB 27.3x27.8 mm, 4x d2.5 mm holes on 23.3x23.8 mm. SSD1315 = SSD1306-compatible. Alt (out of stock): Jixin JX040102-1 C284855, SSD1306 + LDO, 30x29 mm, different hole pattern" (at 66.04 38.10 0) (effects (font (size 1.27 1.27)) (hide yes))) (property "MPN" "PZ254-1-04-Z-C" (at 66.04 38.10 0) (effects (font (size 1.27 1.27)) (hide yes))) (property "LCSC" "C5156431" (at 66.04 38.10 0) (effects (font (size 1.27 1.27)) (hide yes)))
+    (property "Manufacturer" "HCTL" (at 66.04 38.1 0)
       (effects (font (size 1.27 1.27)) (hide yes))
     )
@@
       (effects (font (size 1.27 1.27)) (hide yes))
     )
-    (property "BOM_Note" "J2 = XFCN MF254V-11-04-0743 machined round-hole socket, insulator 3.00+/-0.10 mm (dwg MF254V-11-xx-0743, 2020-04-12); round pins only. OLED module HS96L03W2C03/C5248080 ordered separately (Module_MPN/Module_LCSC). Remove the module's stock square header; fit HCTL PZ254-1-04-Z-C/C5156431 round machined-pin header (Module_Header_*): mating pin d0.50+/-0.03 x 4.13 into J2, solder tail d0.60+/-0.03 through OLED PCB, plastic 3.0 mm (dwg PZ254-1-N-Z-XX-C rev A). Alt Samtec TS-104-G-AA/C3331270 (d0.46 both ends, low stock, insulator height not confirmed). Nominal stack above board top 3.00+3.00+2.65 = 8.65 mm." (at 66.04 38.1 0)
-      (effects (font (size 1.27 1.27)) (hide yes))
-    )
-    (property "Module_Header_MPN" "PZ254-1-04-Z-C" (at 66.04 38.1 0)
-      (effects (font (size 1.27 1.27)) (hide yes))
-    )
-    (property "Module_Header_LCSC" "C5156431" (at 66.04 38.1 0)
-      (effects (font (size 1.27 1.27)) (hide yes))
-    )
-    (property "Module_Header_Manufacturer" "HCTL" (at 66.04 38.1 0)
-      (effects (font (size 1.27 1.27)) (hide yes))
-    )
-    (property "Module_Header_MPN_Alt" "TS-104-G-AA" (at 66.04 38.1 0)
-      (effects (font (size 1.27 1.27)) (hide yes))
-    )
-    (property "Module_Header_LCSC_Alt" "C3331270" (at 66.04 38.1 0)
+    (property "BOM_Note" "1x4 2.54 mm male header, plastic 3.0 mm (HCTL dwg PZ254-1-N-Z-XX-C rev A); no square-pin 1x4 header with 3.0 mm plastic found at LCSC/JLC (all 2.5 mm). OLED module HS96L03W2C03/C5248080 is soldered directly onto this header (module's stock header not used) and is a separate BOM line via Module_MPN/Module_LCSC." (at 66.04 38.1 0)
       (effects (font (size 1.27 1.27)) (hide yes))
     ) (pin "1") (pin "2") (pin "3") (pin "4") (instances (project "TokenKey-RT" (path "/69bcae8e-63e2-488c-b267-fe4af22cfb6e/912f45be-b651-4781-b3b5-bccddac83cec" (reference "J2") (unit 1)))))
@@
 (global_label "LED_A" (shape passive) (at 132.08 73.66 180) (fields_autoplaced yes) (effects (font (size 1.27 1.27)) (justify right)) (property "Intersheetrefs" "${INTERSHEET_REFS}" (at 132.08 73.66 0) (effects (font (size 1.27 1.27)) (hide yes))))
 (global_label "GND" (shape passive) (at 147.32 73.66 0) (fields_autoplaced yes) (effects (font (size 1.27 1.27)) (justify left)) (property "Intersheetrefs" "${INTERSHEET_REFS}" (at 147.32 73.66 0) (effects (font (size 1.27 1.27)) (hide yes))))
-	(text "ASSEMBLY (J2/OLED): remove the OLED module's stock square-pin header and replace it with round machined-pin header HCTL PZ254-1-04-Z-C (LCSC C5156431),\nd0.50 mm mating end into J2 socket, d0.60 mm end soldered through the OLED PCB.\nStack above board top (nominal): socket 3.00 + header plastic 3.00 + OLED module 2.65 = 8.65 mm."
+	(text "ASSEMBLY (J2/OLED): OLED module soldered directly via 3.0 mm header (J2, HCTL PZ254-1-04-Z-C, LCSC C5156431); module stock header not used.\nModule underside 3.0 mm above PCB; OLED top ~5.65 mm (3.0 + 2.65); envelope ~6.65 mm with the 1.0 mm back-side feature."
 		(exclude_from_sim no)
 		(at 25.4 25.4 0)
